File: kiban/EasyEDA/kicad/boardA/boardA.kicad_sch (KiCad schematic)
At the start: 0 parts

Commit message: feat: 基板A / B の回路図を 1 枚に統合し、フットプリント・LCSC 品番・テストポイントを入れる
- 基板B: CHARGER と PROTECTION を手で 1 枚に統合 (KiCad が元データ)
- 基板A: kicad_flat.py で基板B と同じ書き方の 1 枚に作り直し、I2C プルアップ R9/R10 を削除、テストピン J5〜J10 を追加
- assign_footprints.py: LCSC 品番からフットプリントを割り当てる
- testpoints.py: テストパッドを回路図に追加する

Co-Authored-By: Claude Opus 5.5 <noreply@anthropic.com>
Parts:
- added C1: 0.33uF, lcsc:C0603, symbol Device:C_Small
- added C10, C13, C19, C2, C21, C5: 0.1uF, lcsc:C0603, symbol Device:C_Small
- added C11: 10nF, lcsc:C0603, symbol Device:C_Small
- added C12, C22, C23, C24: 10uF, lcsc:C0805, symbol Device:C_Small
- added C14: 47pF, lcsc:C0603, symbol Device:C_Small
- added C15, C16, C17, C18, C8, C9: 22uF, lcsc:C0805, symbol Device:C_Small
- added C20, C3, C7: 1uF, lcsc:C0603, symbol Device:C_Small
- added C4: 0.22uF, lcsc:C0603, symbol Device:C_Small
- added C6: 2.2uF, lcsc:C0603, symbol Device:C_Small
- added J1: MOTHER LEFT, lcsc:HDR-TH_6P-P2.54-V-M, symbol Connector_Generic:Conn_01x06
- added J10: PWR_INT, Connector_PinHeader_2.00mm:PinHeader_1x01_P2.00mm_Vertical, symbol Connector_Generic:Conn_01x01
- added J2: MOTHER RIGHT, lcsc:HDR-TH_6P-P2.54-V-M, symbol Connector_Generic:Conn_01x06
- added J3: TO BOARD B PWR, lcsc:HDR-TH_6P-P2.54-V-M, symbol Connector_Generic:Conn_01x06
- added J4: TO BOARD B SIG, lcsc:HDR-TH_6P-P2.54-V-M, symbol Connector_Generic:Conn_01x06
- added J5: VSYS, Connector_PinHeader_2.00mm:PinHeader_1x01_P2.00mm_Vertical, symbol Connector_Generic:Conn_01x01
- added J6: GND, Connector_PinHeader_2.00mm:PinHeader_1x01_P2.00mm_Vertical, symbol Connector_Generic:Conn_01x01
- added J7: 3V3_MCU, Connector_PinHeader_2.00mm:PinHeader_1x01_P2.00mm_Vertical, symbol Connector_Generic:Conn_01x01
- added J8: 3V3_LED, Connector_PinHeader_2.00mm:PinHeader_1x01_P2.00mm_Vertical, symbol Connector_Generic:Conn_01x01
- added J9: MCU_EN, Connector_PinHeader_2.00mm:PinHeader_1x01_P2.00mm_Vertical, symbol Connector_Generic:Conn_01x01
- added L1: 2.2uH, lcsc:IND-SMD_L4.0-W4.0, symbol Device:L_Small
- added L2: 2.2uH, lcsc:IND-SMD_L7.1-W6.5-P5.60, symbol Device:L_Small
- added R1, R6: 100k, lcsc:R0603, symbol Device:R_Small_US
- added R2: 5.1k, lcsc:R0603, symbol Device:R_Small_US
- added R3: 31.6k, lcsc:R0603, symbol Device:R_Small_US
- added R4, R8: 10k, lcsc:R0603, symbol Device:R_Small_US
- added R5: 93.1k, lcsc:R0603, symbol Device:R_Small_US
- added R7: 20k, lcsc:R0603, symbol Device:R_Small_US
- added U1: LTC2954-1, lcsc:TSOT-23-8_L2.9-W1.6-P0.65-LS2.8-BL, symbol lcsc:LTC2954CTS8-1#TRPBF
- added U2: TPS70933, lcsc:SOT-23-5_L3.0-W1.7-P0.95-LS2.8-BR, symbol lcsc:TPS70933DBVR
- added U3: TPS62933, lcsc:SOT-583-8_L2.1-W1.2-P0.50-LS1.6-BR, symbol lcsc:TPS62933DRLR
- added U4: TPS566238P, lcsc:QFN-9_L2.0-W1.5-P0.50-TL_TPS566238PRQFR, symbol lcsc:TPS566238PRQFR
Connections:
- new net 3V3_AON: C6.1, J1.6 (Pin_6), U2.5 (OUT)
- new net 3V3_LED: C14.1, C15.1, C16.1, C17.1, C18.1, J1.1 (Pin_1), J2.1 (Pin_1), J8.1 (Pin_1), L2.2, R5.1
- new net 3V3_MCU: C8.1, C9.1, J1.3 (Pin_3), J7.1 (Pin_1), L1.2, R1.1, R3.1, R8.1
- new net CHG_INT: J4.4 (Pin_4), R8.2
- new net GND: C1.1, C11.2, C12.2, C13.2, C15.2, C16.2, C17.2, C18.2, C2.2, C20.2, C21.2, C22.2, C23.2, C24.2, C3.2, C4.2, C5.2, C6.2, C7.2, C8.2, C9.2, J1.2 (Pin_2), J2.2 (Pin_2), J2.3 (Pin_3), J3.4 (Pin_4), J3.5 (Pin_5), J3.6 (Pin_6), J4.2 (Pin_2), J4.6 (Pin_6), J6.1 (Pin_1), R4.2, R6.2, R7.2, U1.4 (GND), U2.2 (GND), U3.1 (RT), U3.4 (GND), U4.4 (PGND)
- new net HALL_WAKE: J2.4 (Pin_4), R2.1
- new net I2C_SCL: J1.5 (Pin_5), J4.3 (Pin_3)
- new net I2C_SDA: J1.4 (Pin_4), J4.1 (Pin_1)
- new net LED_EN: J2.6 (Pin_6), R6.1, U4.3 (EN)
- new net L_BST: C19.1, U4.7 (BST)
- new net L_FB: C14.2, R5.2, R7.1, U4.2 (FB)
- new net L_PG: U4.9 (PG)
- new net L_SW: C19.2, L2.1, U4.8 (SW)
- new net L_VCC: C20.1, U4.1 (VCC)
- new net MCU_EN: J9.1 (Pin_1), U1.6 (EN/~{EN}), U3.2 (EN)
- new net M_BST: C10.1, U3.6 (BST)
- new net M_FB: R3.2, R4.1, U3.8 (FB)
- new net M_SS: C11.1, U3.7 (SS)
- new net M_SW: C10.2, L1.1, U3.5 (SW)
- new net ONT: C1.2, U1.3 (ONT)
- new net PB_F: C2.1, R2.2, U1.2 (~{PB})
- new net PDT: C3.1, C4.1, U1.7 (PDT)
- new net PWR_INT: J10.1 (Pin_1), U1.5 (~{INT})
- new net PWR_KILL: J2.5 (Pin_5), R1.2, U1.8 (~{KILL})
- new net VSYS: C12.1, C13.1, C21.1, C22.1, C23.1, C24.1, C5.1, C7.1, J3.1 (Pin_1), J3.2 (Pin_2), J3.3 (Pin_3), J5.1 (Pin_1), U1.1 (VIN), U2.1 (IN), U2.3 (EN), U3.3 (VIN), U4.5 (VIN), U4.6 (VIN)
- no-connect marks 0 -> 2
Other:
- removed sheet LED_IO
- removed sheet POWER
- note added: "3.3 V = 0.8 x (1 + 31.6k / 10k)"
- note added: "3V3_AON：北極の DRV5032FC だけに給電（待機電流 1.4 uA）"
- note added: "EN（MCU_EN）は U3 の EN に直結（外付けプルアップなし。U3 の内部プルアップ 0.7 uA）"
- note added: "HALL_WAKE：北極 DRV5032FC（磁石で L）"
- note added: "I2C 4.7k、CHG_INT 10k"
- note added: "J1：左（3V3_LED_L / GND_L / 3V3_MCU / SDA / SCL / 3V3_AON）"
- note added: "J2：右（3V3_LED_R / GND_R / GND_SYS / HALL_WAKE / PWR_KILL / LED_EN）"
- note added: "J3 / J4 は基板B の J_AB1 / J_AB2 と同じピン配置"
- note added: "KILL は 3V3_MCU へプルアップ"
- note added: "LED 用 3.3 V 降圧 U4 TPS566238P（6 A、LED_EN で ON）"
- note added: "LED_EN：GND へ 100k（MCU 起動前は OFF）"
- note added: "L_PG：テストパッドへ（任意）"
- note added: "MCU 用 3.3 V 降圧 U3 TPS62933（1.2 MHz、LTC2954 が EN を制御）"
- note added: "ON 長押し 約 2.15 s"
- note added: "PWR_INT はテストパッドへ（任意）"
- note added: "PWR_KILL の 100k は POWER ページ"
- note added: "RT = GND：1.2 MHz"
- note added: "mother-ring 接続（1x6 × 2、左右の張り出し）"
- note added: "テストパッド（直径 1.0 mm、部品なし。コネクタのピンで測れないネットだけ）"
- note added: "プルアップ（3V3_MCU、基板A に集約）"
- note added: "出力 = 0.6 x (1 + 93.1k / 20k) = 3.39 V"
- note added: "基板B 接続（ピンヘッダ 1x6 × 2）"
- note added: "常時オン 3.3 V U2 TPS70933"
- note added: "強制 OFF 約 7.9 s（1 + 0.22 uF）"
- note added: "電源 ON/OFF U1 LTC2954-1（磁石の長押し）"
- note added: "（WS2812C の下限 3.3 V に余裕。実測後に R5 を調整）"
- note removed: "boardA（power-2s-xiao）— EasyEDA から自動生成。編集は EasyEDA で行う"
